File: rev_a/bus_raspberry_pi.sch (KiCad schematic (older format))
At the start: 39 parts, among them J1 TERMINATE_JUMPER, Q1 FQP47P06, SW1 2_LEAD_PUSH_BUTTON, U1 74x05, U2 74X08, U3 MCP2562, U5 ATMEGA324_DIP40, X1 16MHz, X2 OSHW_LOGO

Commit message: Next iteration of schematic; started board layout.
Parts:
- removed N9: RASPI_CONNECTOR, symbol RASPI_CONNECTOR
- removed R1, R4: 100K, symbol R_VERT
- removed R13: 22K 1%, symbol R_VERT
- removed R14: 33K 1%, symbol R_VERT
- removed unit 3 of U2
- added C4, C5, C6, C7: .1uF, symbol C_VERT
- added D2: LED, symbol LED
- added J2: LED_JUMPER, symbol LED_JUMPER
- added N9: RASPI_CONNECTOR_40, symbol RASPI_CONNECTOR_40
- added R12, R17, R6, R8: 33K 1%, symbol R_VERT
- added R15: 100K, symbol R_VERT
- added R16, R5, R7: 22K 1%, symbol R_VERT
- added R18, R19: 470, symbol R_VERT
- N7: value ARD_SPI_HEADER -> AVR_ISP_HEADER
- N8: value AVR_JTAG_CONNECTOR -> BHR-10-HUA
- R1: renamed from R5; value 10K -> 22K 1%
- R11: value 100K -> 22K 1%
- R2: value 100K -> 33K 1%
- SW1: value 2_LEAD_PUSH_BUTTON -> MJTP1243
- renumbered R8 to R10, R9 to R13, R10 to R14, R6 to R4, R7 to R9, U3 to U2, U2 to U3, U5 to U4
Connections:
- net +5V: now also C4.1, C5.1, C6.1, C7.1, N9.2 (5V), N9.4 (5V), R16.2, R19.2, R5.2, R7.2; no longer R11.2, R2.2
- net GND: now also R2.1, C4.2, C5.2, C6.2, C7.2, D2.-, N9.14 (GND), N9.20 (GND), N9.25 (GND), N9.30 (GND), N9.34 (GND), N9.39 (GND), N9.9 (GND), R12.1, R15.1, R17.1, R6.1, R8.1
- net XTAL2: now reaches C1.1, U4.12 (XTAL2), X1.1
- net XTAL1: now reaches C2.1, U4.13 (XTAL1), X1.2
- net RXD0: now reaches U3.3, U4.14 (PD0/RXD0)
- net at N2.5 (RXD), R11.1: now also U3.4, R12.2; no longer U3.5, U4.15 (PD1/TXD0)
- net RXD1: now reaches U2.1 (TXD), U4.16 (PD2/RXD1/INT0)
- net TXD1: now reaches U2.4 (RXD), U4.17 (PD3/TXD1/INT1)
- net TCK: now reaches N8.1 (TCK), U4.24 (PC2/TCK)
- net TMS: now reaches N8.5 (TMS), U4.25 (PC3/TMS)
- net TDO: now reaches N8.3 (TDO), U4.26 (PC4/TDO)
- net TDI: now reaches N8.9 (TDI), U4.27 (PC5/TDI)
- net MOSI: now reaches N7.4 (MOSI), U4.6 (PB5/MOSI)
- net MISO: now reaches N7.1 (MISO), U4.7 (PB6/MISO)
- net SCK: now reaches N7.3 (SCK), U4.8 (PB7/SCK)
- net SCK: now also R18.2
- net ~RESET: now reaches C3.2, D1.+, N7.5 (~RESET), N8.6 (~NRST), R10.1, SW1.2, U1.6, U4.9 (~RESET)
- net at U1.5: now also N9.26 (GPIO7_CE1), R15.2
- net at N2.6 (~RTS), U1.1: now also R5.1, R6.2
- net at N3.5 (RXD), U3.2: now also N9.8 (GPIO14_TXD), R16.1, R17.2
- net at N3.4 (TXD), R1.1: now also R2.2, U3.5; no longer U3.4
- net at N2.4 (TXD), U3.1: now also R7.1, R8.2; no longer R2.1
- net at R13.1, R14.2: now also N9.10 (GPIO15_RXD)
- new net: D2.+, J2.3 (LED), J2.4 (LED)
- new net: J2.1 (POWER), R19.1
- new net: J2.2 (D13), R18.1
- new net TXD0: R11.2, U4.15 (PD1/TXD0)
- no-connect marks 47 -> 63
Other:
- note added: "5V @ 1.5A DC/DC Converter"
- note added: "6-pin AVR ISP\nConnector"
- note added: "AVR JTAG Connector"
- note added: "BUS HEADER"
- note added: "Bus Transceiver"
- note added: "Filter Capacitors"
- note added: "Jumper 1-3: Power LED\nJumper 2-4: D13 LED\nJumper 3-4: No LED"
- note added: "Note: U1, U3 have ground connected\nto pin 7 and VCC connected to pin 14."
- note added: "Reset Circuitry"
- note removed: "Note: U1, U2, U3 have ground connected\nto pin 7 and VCC connected to pin 14."
- moved on the sheet: H1, H2, H3, H4, N6, N7, N8, R1, R13, R14, R4, U1A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

Commit message: Layed out PCB.
Parts:
- removed C4: .1uF, symbol C_VERT
- removed R1, R11, R13, R16, R5, R7: 22K 1%, symbol R_VERT
- removed R12, R14, R17, R2, R6, R8: 33K 1%, symbol R_VERT
- removed R15, R4: 100K, symbol R_VERT
- removed R9: 10K, symbol R_VERT
- removed U1: 74x05, symbol 74x05
- added C7: .1uF, symbol C_VERT
- added C8: .1uF, symbol C_HORIZ
- added N8: SERIAL_CONNECTOR, symbol SERIAL_CONNECTOR
- added R1: 22K, symbol R_VERT_SIP8
- added R2: 33K, symbol R_VERT_SIP8
- added unit 1 of U1
- added unit 4 of U1
- U1: renamed from U3; value 74X08 -> 74HCT08
- renumbered C5 to C3, C6 to C4, C7 to C5, C3 to C6, N4 to N1, N9 to N10, N5 to N2, N1 to N3, N2 to N4, N3 to N5, N8 to N9, R10 to R4, R18 to R5, R19 to R6, U4 to U3
Connections:
- net +5V: now also C7.1, R1.1, R1.1, R1.1, R1.1, R1.1, U1.1, U1.13, U1.14 (VCC), U1.14 (VCC)
- net GND: now also C7.2, N8.1 (GND), R2.1, R2.1, R2.1, R2.1, R2.1, R2.1, R2.1, U1.7 (GND), U1.7 (GND)
- net RXD0: now also U1.6; no longer U1.3
- net TXD0: now also R1.1
- net ~RESET: now also C8.1; no longer N9.6 (~NRST)
- net BAT+: now reaches N1.1 (+), N2.1 (+), Q1.D
- net at N10.26 (GPIO7_CE1): now also N8.4 (~RESET), R1.7, R2.7, U1.12
- net at N4.6 (~RTS): now also R1.3, R2.3, U1.2
- net at C6.1: now also U1.3
- net CANL: now reaches J1.2 (COM), N3.6 (CANL), U2.6 (CANL)
- net CANH: now reaches N3.5 (CANH), R3.1, U2.7 (CANH)
- net at N5.4 (TXD): now also U1.10, R1.2, R2.2; no longer U1.5
- net at N10.8 (GPIO14_TXD), N5.5 (RXD): now also U1.5, N8.2 (TXD), R1.8, R2.8; no longer U1.2
- net at N4.4 (TXD): now also U1.4, R1.4, R2.4; no longer U1.1
- net at N4.5 (RXD): now also U1.9, R1.5, R2.5; no longer U1.4
- net at N10.10 (GPIO15_RXD): now also N8.3 (RXD), R1.6, R2.6
- new net: C8.2, N9.6 (~NRST), U1.11
- new net: R1.1, U1.8
Other:
- note added: "Note: U1 has ground connected to\npin 7 and VCC connected to pin 14."
- note removed: "Note: U1, U3 have ground connected\nto pin 7 and VCC connected to pin 14."
- moved on the sheet: C3, C4, C5, N1, N2, U2
