File: rev_b/bus_raspberry_pi.kicad_pcb (KiCad board)
At the start: 2 copper layers, 100 x 50 mm, 47 parts, among them J1 TERMINATE_JUMPER, J2 LED_JUMPER, SW1 MJTP1243, U1 MCP7940, U2 74HCT08, U3 MCP2562, U4 L78L05AC, U5 ATMEGA324_DIP40, U6 L78L33AC, X1 16MHz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

Commit message: Revision B is ready for manufacture.
Parts:
- removed N10: BBB_P9_HEADER, bus_beaglebone:Pin_Header_Straight_2x23
- removed N11, N12, N13: KEY2, bus_beaglebone:Pin_Header_Straight_1x02
- removed R7: 4K7, bus_beaglebone:Resistor_Horizontal__400
- added C12: .1uF, bus_raspberry_pi:Capacitor3MMDiscRM2.5, F.Cu at (148.6, 108.0)
- added C13: .1uF, bus_raspberry_pi:Capacitor3MMDiscRM2.5, F.Cu at (125.7, 111.1)
- added N1: RASPI_CONNECTOR_40, bus_raspberry_pi:Pin_Header_Straight_2x20, F.Cu at (128.3, 102.9)
- added U7: MCP24XX32A, bus_raspberry_pi:DIP-8__300, F.Cu at (132.7, 111.1)
- BAT1: footprint bus_beaglebone:10MM_BATTERY -> bus_raspberry_pi:10MM_BATTERY
- C1, C10, C11, C2, C3, C4, C5, C6, C7, C8, C9: footprint bus_beaglebone:Capacitor3MMDiscRM2.5 -> bus_raspberry_pi:Capacitor3MMDiscRM2.5
- D1: footprint bus_beaglebone:Diode_DO-41_SOD81_Horizontal_RM10 -> bus_raspberry_pi:Diode_DO-41_SOD81_Horizontal_RM10
- D2: footprint bus_beaglebone:T1_LED -> bus_raspberry_pi:T1_LED
- H1, H2, H3, H4: footprint bus_beaglebone:MountingHole_3mm -> bus_raspberry_pi:MountingHole_3mm
- H5: footprint bus_beaglebone:OSHW_LOGO_250mil -> bus_raspberry_pi:OSHW_LOGO_250mil
- J1: footprint bus_beaglebone:Pin_Header_Straight_1x03 -> bus_raspberry_pi:Pin_Header_Straight_1x03
- J2: footprint bus_beaglebone:Pin_Header_Straight_2x02 -> bus_raspberry_pi:Pin_Header_Straight_2x02
- N3, N9: footprint bus_beaglebone:Pin_Header_Straight_2x05_Shrouded -> bus_raspberry_pi:Pin_Header_Straight_2x05_Shrouded
- N4, N5, R2: footprint bus_beaglebone:Pin_Header_Straight_1x06 -> bus_raspberry_pi:Pin_Header_Straight_1x06
- N7: footprint bus_beaglebone:Pin_Header_Straight_2x03 -> bus_raspberry_pi:Pin_Header_Straight_2x03
- N8: footprint bus_beaglebone:Pin_Header_Straight_1x04 -> bus_raspberry_pi:Pin_Header_Straight_1x04
- R1, R3, R4, R5: footprint bus_beaglebone:Resistor_Horizontal__400 -> bus_raspberry_pi:Resistor_Horizontal__400
- R6: value 4K7 -> 3K9_SIP5; footprint bus_beaglebone:Resistor_Horizontal__400 -> bus_raspberry_pi:Pin_Header_Straight_1x05
- SW1: footprint bus_beaglebone:Button_6.5MM -> bus_raspberry_pi:Button_6.5MM
- U1, U3: footprint bus_beaglebone:DIP-8__300 -> bus_raspberry_pi:DIP-8__300
- U2: footprint bus_beaglebone:DIP-14__300 -> bus_raspberry_pi:DIP-14__300
- U4, U6: footprint bus_beaglebone:TO92_123 -> bus_raspberry_pi:TO92_123
- U5: footprint bus_beaglebone:DIP-40__600 -> bus_raspberry_pi:DIP-40__600
- X1: footprint bus_beaglebone:Crystal_HC49-U_Vertical -> bus_raspberry_pi:Crystal_HC49-U_Vertical
- X2: footprint bus_beaglebone:RTC_CRYSTAL -> bus_raspberry_pi:RTC_CRYSTAL
- moved N8 30.7 mm to (161.3, 101.6)
- moved R6 27.1 mm to (138.4, 118.7), turned to 0 degrees
- moved X2 2.62 mm to (142.2, 110.5)
Connections:
- C11 pad 1: VCC -> +3.3V
- C3 pad 1: VCC -> +3.3V
- C4 pad 1: VCC -> +3.3V
- C5 pad 1: VCC -> +3.3V
- C7 pad 1: VCC -> +3.3V
- D1 pad -: VCC -> +3.3V
- H1 pad 1: GND -> (no net)
- H2 pad 1: GND -> (no net)
- H3 pad 1: GND -> (no net)
- H4 pad 1: GND -> (no net)
- N7 pad 2: VCC -> +3.3V
- N8 pad 4: Net-(N10-Pad27) -> Net-(N1-Pad24)
- N9 pad 4: VCC -> +3.3V
- R2 pad 1: VCC -> +3.3V
- R2 pad 6: (no net) -> Net-(N1-Pad24)
- R3 pad 2: VCC -> +3.3V
- R5 pad 2: VCC -> +3.3V
- R6 pad 1: Net-(R6-Pad1) -> +3.3V
- R6 pad 2: VCC -> Net-(R6-Pad2)
- U1 pad 5: Net-(R6-Pad1) -> Net-(R6-Pad2)
- U1 pad 6: Net-(R7-Pad1) -> Net-(R6-Pad3)
- U1 pad 8: VCC -> +3.3V
- U2 pad 1: VCC -> +3.3V
- U2 pad 10: VCC -> +3.3V
- U2 pad 14: VCC -> +3.3V
- U2 pad 9: Net-(N10-Pad27) -> Net-(N1-Pad24)
- U3 pad 5: VCC -> +3.3V
- U5 pad 10: VCC -> +3.3V
- U5 pad 22: Net-(R7-Pad1) -> Net-(R6-Pad3)
- U5 pad 23: Net-(R6-Pad1) -> Net-(R6-Pad2)
- U5 pad 30: VCC -> +3.3V
- U6 pad 1: VCC -> +3.3V
Routing:
- net +3.3V: track 0.00 -> 233.9 mm
- net VCC: track 219.9 -> 0.00 mm
- net GND: track 123.1 -> 225.8 mm, vias 10 -> 22
- net Net-(N1-Pad24): track 0.00 -> 97.1 mm, vias 0 -> 2
- net Net-(N10-Pad27): track 71.2 -> 0.00 mm, vias 1 -> 0
- net Net-(N1-Pad27): track 0.00 -> 42.7 mm
- net Net-(N1-Pad28): track 0.00 -> 36.7 mm
- net Net-(R6-Pad2): track 0.00 -> 32.5 mm
- net Net-(R6-Pad1): track 30.7 -> 0.00 mm
- net Net-(R6-Pad3): track 0.00 -> 25.2 mm
- net Net-(R7-Pad1): track 17.6 -> 0.00 mm
- net /~RESET: track 118.0 -> 104.5 mm, vias 0 -> 2
- net Net-(N1-Pad10): track 81.5 -> 68.8 mm, vias 1 -> 2
- net /TDI: track 40.6 -> 41.8 mm
- net Net-(U1-Pad1): track 4.48 -> 5.01 mm
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Other:
- board text added: "+"
- board text added: "-"
- board text added: "BUS RASPBERRY PI REV. B 13JAN2014 (C) 2015 GRAMLICH"
- board text added: "BUS RASPBERRY PI REV. B 13JAN2015 (C) 2015 GRAMLICH"
- board text removed: "BUS BEAGLEBON REV. D 11JAN2014 (C) 2015 GRAMLICH"
- board text removed: "BUS BEAGLEBONE REV. D 11JAN2015 (C) 2015 GRAMLICH"
