File: rev_c/bus_raspberry_pi.kicad_pcb (KiCad board)
At the start: 2 copper layers, 100 x 50 mm, 46 parts, among them J1 TERMINATE_JUMPER, J2 LED_JUMPER, SW1 MJTP1243, U1 MCP7940, U2 74HCT08, U3 MCP2562, U4 L78L05AC, U5 ATMEGA324_DIP40, U6 L78L33AC, U7 MCP24XX32A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

Commit message: Changed from B=>C.  Flipped N1.
Parts:
- N1: moved to B.Cu
Routing:
- net GND: track 225.8 -> 201.8 mm, vias 22 -> 23
- net Net-(N1-Pad27): track 42.7 -> 34.9 mm
- net Net-(N1-Pad28): track 36.7 -> 40.3 mm
- net Net-(N1-Pad10): track 68.8 -> 71.0 mm, vias 2 -> 3
- net Net-(N1-Pad8): track 71.0 -> 69.9 mm, vias 0 -> 1
- net Net-(N1-Pad24): track 97.1 -> 96.4 mm
Other:
- board text added: "BUS RASPBERRY PI REV. B 1FEB2015 (C) 2015 GRAMLICH"
- board text added: "BUS RASPBERRY PI REV. C 1FEB2015 (C) 2015 GRAMLICH"
- board text removed: "BUS RASPBERRY PI REV. B 13JAN2014 (C) 2015 GRAMLICH"
- board text removed: "BUS RASPBERRY PI REV. B 13JAN2015 (C) 2015 GRAMLICH"

Commit message: Minor changes to Rev. C.
Parts:
- removed C10: .1uF, bus_raspberry_pi:Capacitor3MMDiscRM2.5
- added J3: RESET_SEL, bus_raspberry_pi:Pin_Header_Straight_1x03, F.Cu at (114.3, 145.4)
- added R7: 100K, bus_raspberry_pi:Resistor_Horizontal__400, F.Cu at (165.1, 116.8)
- U2: value 74HCT08 -> 74HC08
Connections:
- C11 pad 1: +3.3V -> VCC
- C12 pad 1: +3.3V -> VCC
- C13 pad 1: +3.3V -> VCC
- C3 pad 1: +3.3V -> VCC
- C4 pad 1: +3.3V -> VCC
- C5 pad 1: +3.3V -> VCC
- C7 pad 1: +3.3V -> VCC
- D1 pad -: +3.3V -> VCC
- N7 pad 2: +3.3V -> VCC
- N7 pad 5: /~RESET -> Net-(J3-Pad2)
- N9 pad 4: +3.3V -> VCC
- R2 pad 1: +3.3V -> VCC
- R3 pad 2: +3.3V -> VCC
- R5 pad 2: +3.3V -> VCC
- R6 pad 1: +3.3V -> VCC
- U1 pad 8: +3.3V -> VCC
- U2 pad 1: +3.3V -> Net-(R7-Pad1)
- U2 pad 10: +3.3V -> VCC
- U2 pad 14: +3.3V -> VCC
- U2 pad 8: Net-(C10-Pad2) -> (no net)
- U3 pad 5: +3.3V -> VCC
- U5 pad 10: +3.3V -> VCC
- U5 pad 3: (no net) -> Net-(J3-Pad1)
- U5 pad 30: +3.3V -> VCC
- U6 pad 1: +3.3V -> VCC
- U7 pad 8: +3.3V -> VCC
Routing:
- net VCC: track 0.00 -> 240.8 mm
- net +3.3V: track 233.9 -> 0.00 mm
- net GND: track 201.8 -> 405.4 mm, vias 23 -> 53
- net Net-(C10-Pad2): track 47.0 -> 0.00 mm
- net Net-(J3-Pad1): track 0.00 -> 12.9 mm
- net Net-(R7-Pad1): track 0.00 -> 11.8 mm
- net Net-(J3-Pad2): track 0.00 -> 11.2 mm
- net /~RESET: track 104.5 -> 99.4 mm
- net Net-(U3-Pad8): track 43.7 -> 44.8 mm
- net Net-(C6-Pad1): track 30.1 -> 31.2 mm
- net /TDO: track 31.6 -> 31.1 mm
Other:
- board text added: "(C) 2015 GRAMLICH"
- board text added: "BUS RASPBERRY PI REV. C 8FEB2015"
- board text added: "BUS RASPBERRY PI REV. C 8FEB2015 (C) 2015 GRAMLICH"
- board text added: "PGM"
- board text added: "RST"
- board text removed: "BUS RASPBERRY PI REV. B 1FEB2015 (C) 2015 GRAMLICH"
- board text removed: "BUS RASPBERRY PI REV. C 1FEB2015 (C) 2015 GRAMLICH"
